File: hw/SolderingInduction.kicad_sch (KiCad schematic)
At the start: 54 parts, among them J1 C116159, J3 RBP_GPIO_CONN, SW1 SW_Push, SW2 SW_Push, SW3 SW_Push, SW4 SW_Push, SW5 SW_Push, SW6 SW_Push, SW7 SW_Push, SW8 SW_Push, U1 ASM1117-3.3, U3 WQ25JVS, U4 RP2040, Y1 X322512MMB4SI

Commit message: Repo cleanup
Parts:
- SW1: value SW_Push -> DOWN
- SW2: value SW_Push -> START
- SW3: value SW_Push -> LEFT
- SW4: value SW_Push -> B
- SW5: value SW_Push -> UP
- SW6: value SW_Push -> A
- SW7: value SW_Push -> RIGHT
- SW8: value SW_Push -> SELECT
Other:
- moved on the sheet: FID1, FID2, FID3, J3A, J3B, SW1, SW2, SW3, SW4, SW5, SW6, SW7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
