File: autotesting/hw/SolderingInduction.kicad_sch (KiCad schematic)
At the start: 54 parts, among them J1 C116159, J3 RBP_GPIO_CONN, SW1 DOWN, SW2 START, SW3 LEFT, SW4 B, SW5 UP, SW6 A, SW7 RIGHT, SW8 SELECT, U1 ASM1117-3.3, U3 WQ25JVS, U4 RP2040, Y1 X322512MMB4SI

Commit message: General autotest rig schematic
Parts:
- removed C1, C11, C8: 1μF, Capacitor_SMD:C_0805_2012Metric, symbol Device:C_Small
- removed C10, C12, C13, C14, C15, C16, C17, C18, C7, C9: 100nF, Capacitor_SMD:C_0805_2012Metric, symbol Device:C_Small
- removed C2, C3: 10${uF}, Capacitor_SMD:C_1206_3216Metric, symbol Device:C_Small
- removed C4: 1${uF}, Capacitor_SMD:C_0805_2012Metric, symbol Device:C_Small
- removed C5, C6: 14pF, Capacitor_SMD:C_0805_2012Metric, symbol Device:C_Small
- removed F1: C261953, Fuse:Fuse_1206_3216Metric, symbol Device:Polyfuse
- removed FID1: 0,1, Fiducial:Fiducial_1mm_Mask2mm, symbol Mechanical:Fiducial
- removed FID2: 0,0, Fiducial:Fiducial_1mm_Mask2mm, symbol Mechanical:Fiducial
- removed FID3: 1,0, Fiducial:Fiducial_1mm_Mask2mm, symbol Mechanical:Fiducial
- removed J1: C116159, Connector_USB:USB_C_Receptacle_Palconn_UTC16-G, symbol Connector:USB_C_Receptacle_USB2.0
- removed LED1: WS2812B, LED_SMD:LED_WS2812B_PLCC4_5.0x5.0mm_P3.2mm, symbol LED:WS2812B
- removed R1, R5: 5.1kΩ, Resistor_SMD:R_0805_2012Metric, symbol Device:R_Small
- removed R2, R3: 27Ω, Resistor_SMD:R_0603_1608Metric, symbol Device:R_Small
- removed R6: 10kΩ, Resistor_SMD:R_0805_2012Metric, symbol Device:R_Small
- removed SW1: DOWN, 0:SW_TSC016XXXXXXX_4.5x3.0_H2.75, symbol Switch:SW_Push
- removed SW2: START, 0:SW_TSC016XXXXXXX_4.5x3.0_H2.75, symbol Switch:SW_Push
- removed SW3: LEFT, 0:SW_TSC016XXXXXXX_4.5x3.0_H2.75, symbol Switch:SW_Push
- removed SW4: B, 0:SW_TSC016XXXXXXX_4.5x3.0_H2.75, symbol Switch:SW_Push
- removed SW5: UP, 0:SW_TSC016XXXXXXX_4.5x3.0_H2.75, symbol Switch:SW_Push
- removed SW6: A, 0:SW_TSC016XXXXXXX_4.5x3.0_H2.75, symbol Switch:SW_Push
- removed SW7: RIGHT, 0:SW_TSC016XXXXXXX_4.5x3.0_H2.75, symbol Switch:SW_Push
- removed SW8: SELECT, 0:SW_TSC016XXXXXXX_4.5x3.0_H2.75, symbol Switch:SW_Push
- removed TP1: MCU 3v3, 0:Testpoint_Custom, symbol Connector:TestPoint_Flag
- removed TP10: LDO_{VIN}, 0:Testpoint_Custom, symbol Connector:TestPoint_Flag
- removed TP11: SWD_3V3, 0:Testpoint_Custom, symbol 4ms_Connector:TestPoint_Small
- removed TP12: ~{CS}, 0:Testpoint_Custom, symbol Connector:TestPoint_Flag
- removed TP2: MCU 1v2, 0:Testpoint_Custom, symbol Connector:TestPoint_Flag
- removed TP3: RUN, 0:Testpoint_Custom, symbol 4ms_Connector:TestPoint_Small
- removed TP4: SWCLK, 0:Testpoint_Custom, symbol 4ms_Connector:TestPoint_Small
- removed TP5: LED DATA, 0:Testpoint_Custom, symbol Connector:TestPoint_Flag
- removed TP6: SWD, 0:Testpoint_Custom, symbol 4ms_Connector:TestPoint_Small
- removed TP7: RUN_GND, 0:Testpoint_Custom, symbol 4ms_Connector:TestPoint_Small
- removed TP8: VBUS, 0:Testpoint_Custom, symbol Connector:TestPoint_Flag
- removed TP9: LDO_{VOUT}, 0:Testpoint_Custom, symbol Connector:TestPoint_Flag
- removed U1: ASM1117-3.3, Package_TO_SOT_SMD:SOT-223-3_TabPin2, symbol Regulator_Linear:AMS1117CD-3.3
- removed U3: WQ25JVS, 0:FLASH-SOIC-8, symbol Memory_Flash:W25Q128JVS
- removed U4: RP2040, Package_DFN_QFN:QFN-56-1EP_7x7mm_P0.4mm_EP3.2x3.2mm, symbol MCU_RaspberryPi:RP2040
- removed Y1: X322512MMB4SI, Crystal:Crystal_SMD_3225-4Pin_3.2x2.5mm, symbol Device:Crystal_GND24_Small
- added U?: MSP430F5309IRGC, Package_DFN_QFN:Texas_S-PVQFN-N64_EP4.25x4.25mm, symbol MCU_Texas_MSP430:MSP430F5309IRGC
Connections:
- net VBUS renamed LDO_{VIN}
- no-connect marks 4 -> 0
Other:
- added sheet Untitled Sheet (testchannel.kicad_sch)
- added sheet Untitled Sheet1 (testchannel.kicad_sch)
- added sheet Untitled Sheet2 (testchannel.kicad_sch)
- added sheet Untitled Sheet3 (testchannel.kicad_sch)
- added sheet Untitled Sheet4 (testchannel.kicad_sch)
- moved on the sheet: J3A, J3B

Commit message: Revert "General autotest rig schematic"
This reverts commit edc100e629294de22c7f368bf0c62424b6d2474e.
Parts:
- removed U?: MSP430F5309IRGC, Package_DFN_QFN:Texas_S-PVQFN-N64_EP4.25x4.25mm, symbol MCU_Texas_MSP430:MSP430F5309IRGC
- added C1, C11, C8: 1μF, Capacitor_SMD:C_0805_2012Metric, symbol Device:C_Small
- added C10, C12, C13, C14, C15, C16, C17, C18, C7, C9: 100nF, Capacitor_SMD:C_0805_2012Metric, symbol Device:C_Small
- added C2, C3: 10${uF}, Capacitor_SMD:C_1206_3216Metric, symbol Device:C_Small
- added C4: 1${uF}, Capacitor_SMD:C_0805_2012Metric, symbol Device:C_Small
- added C5, C6: 14pF, Capacitor_SMD:C_0805_2012Metric, symbol Device:C_Small
- added F1: C261953, Fuse:Fuse_1206_3216Metric, symbol Device:Polyfuse
- added FID1: 0,1, Fiducial:Fiducial_1mm_Mask2mm, symbol Mechanical:Fiducial
- added FID2: 0,0, Fiducial:Fiducial_1mm_Mask2mm, symbol Mechanical:Fiducial
- added FID3: 1,0, Fiducial:Fiducial_1mm_Mask2mm, symbol Mechanical:Fiducial
- added J1: C116159, Connector_USB:USB_C_Receptacle_Palconn_UTC16-G, symbol Connector:USB_C_Receptacle_USB2.0
- added LED1: WS2812B, LED_SMD:LED_WS2812B_PLCC4_5.0x5.0mm_P3.2mm, symbol LED:WS2812B
- added R1, R5: 5.1kΩ, Resistor_SMD:R_0805_2012Metric, symbol Device:R_Small
- added R2, R3: 27Ω, Resistor_SMD:R_0603_1608Metric, symbol Device:R_Small
- added R6: 10kΩ, Resistor_SMD:R_0805_2012Metric, symbol Device:R_Small
- added SW1: DOWN, 0:SW_TSC016XXXXXXX_4.5x3.0_H2.75, symbol Switch:SW_Push
- added SW2: START, 0:SW_TSC016XXXXXXX_4.5x3.0_H2.75, symbol Switch:SW_Push
- added SW3: LEFT, 0:SW_TSC016XXXXXXX_4.5x3.0_H2.75, symbol Switch:SW_Push
- added SW4: B, 0:SW_TSC016XXXXXXX_4.5x3.0_H2.75, symbol Switch:SW_Push
- added SW5: UP, 0:SW_TSC016XXXXXXX_4.5x3.0_H2.75, symbol Switch:SW_Push
- added SW6: A, 0:SW_TSC016XXXXXXX_4.5x3.0_H2.75, symbol Switch:SW_Push
- added SW7: RIGHT, 0:SW_TSC016XXXXXXX_4.5x3.0_H2.75, symbol Switch:SW_Push
- added SW8: SELECT, 0:SW_TSC016XXXXXXX_4.5x3.0_H2.75, symbol Switch:SW_Push
- added TP1: MCU 3v3, 0:Testpoint_Custom, symbol Connector:TestPoint_Flag
- added TP10: LDO_{VIN}, 0:Testpoint_Custom, symbol Connector:TestPoint_Flag
- added TP11: SWD_3V3, 0:Testpoint_Custom, symbol 4ms_Connector:TestPoint_Small
- added TP12: ~{CS}, 0:Testpoint_Custom, symbol Connector:TestPoint_Flag
- added TP2: MCU 1v2, 0:Testpoint_Custom, symbol Connector:TestPoint_Flag
- added TP3: RUN, 0:Testpoint_Custom, symbol 4ms_Connector:TestPoint_Small
- added TP4: SWCLK, 0:Testpoint_Custom, symbol 4ms_Connector:TestPoint_Small
- added TP5: LED DATA, 0:Testpoint_Custom, symbol Connector:TestPoint_Flag
- added TP6: SWD, 0:Testpoint_Custom, symbol 4ms_Connector:TestPoint_Small
- added TP7: RUN_GND, 0:Testpoint_Custom, symbol 4ms_Connector:TestPoint_Small
- added TP8: VBUS, 0:Testpoint_Custom, symbol Connector:TestPoint_Flag
- added TP9: LDO_{VOUT}, 0:Testpoint_Custom, symbol Connector:TestPoint_Flag
- added U1: ASM1117-3.3, Package_TO_SOT_SMD:SOT-223-3_TabPin2, symbol Regulator_Linear:AMS1117CD-3.3
- added U3: WQ25JVS, 0:FLASH-SOIC-8, symbol Memory_Flash:W25Q128JVS
- added U4: RP2040, Package_DFN_QFN:QFN-56-1EP_7x7mm_P0.4mm_EP3.2x3.2mm, symbol MCU_RaspberryPi:RP2040
- added Y1: X322512MMB4SI, Crystal:Crystal_SMD_3225-4Pin_3.2x2.5mm, symbol Device:Crystal_GND24_Small
Connections:
- net $.GPIO1: now also SW4.2, U4.3 (GPIO1)
- net $.GPIO10: now also U4.13 (GPIO10)
- net $.GPIO11: now also SW5.2, U4.14 (GPIO11)
- net $.GPIO12: now also U4.15 (GPIO12)
- net $.GPIO13: now also U4.16 (GPIO13)
- net $.GPIO14: now also U4.17 (GPIO14)
- net $.GPIO15: now also U4.18 (GPIO15)
- net $.GPIO16: now also U4.27 (GPIO16)
- net $.GPIO17: now also U4.28 (GPIO17)
- net $.GPIO18: now also U4.29 (GPIO18)
- net $.GPIO19: now also U4.30 (GPIO19)
- net $.GPIO2: now also SW2.2, U4.4 (GPIO2)
- net $.GPIO20: now also U4.31 (GPIO20)
- net $.GPIO21: now also U4.32 (GPIO21)
- net $.GPIO22: now also U4.34 (GPIO22)
- net $.GPIO23: now also U4.35 (GPIO23)
- net $.GPIO24: now also U4.36 (GPIO24)
- net $.GPIO25: now also LED1.4 (DIN), TP5.1, U4.37 (GPIO25)
- net $.GPIO26: now also U4.38 (GPIO26_ADC0)
- net $.GPIO27: now also U4.39 (GPIO27_ADC1)
- net $.GPIO28: now also U4.40 (GPIO28_ADC2)
- net $.GPIO29: now also U4.41 (GPIO29_ADC3)
- net $.GPIO3: now also SW8.2, U4.5 (GPIO3)
- net $.GPIO4: now also SW1.2, U4.6 (GPIO4)
- net $.GPIO5: now also SW3.2, U4.7 (GPIO5)
- net $.GPIO6: now also U4.8 (GPIO6)
- net $.GPIO8: now also SW7.2, U4.11 (GPIO8)
- net $.GPIO9: now also U4.12 (GPIO9)
- net +3V3: now also C11.1, C12.1, C13.1, C14.1, C15.1, C16.1, C17.1, C18.1, C3.1, C4.1, C7.1, R6.2, TP1.1, TP11.1, TP9.1, U1.2 (VO), U3.8 (VCC), U4.1 (IOVDD), U4.10 (IOVDD), U4.22 (IOVDD), U4.33 (IOVDD), U4.42 (IOVDD), U4.43 (ADC_AVDD), U4.44 (VREG_IN), U4.48 (USB_VDD), U4.49 (IOVDD)
- net GND: now also C1.2, C10.2, C11.2, C12.2, C13.2, C14.2, C15.2, C16.2, C17.2, C18.2, C2.2, C3.2, C4.2, C5.2, C6.2, C7.2, C8.2, C9.2, J1.A1 (GND), J1.A12 (GND), J1.B1 (GND), J1.B12 (GND), LED1.3 (VSS), R1.2, R5.2, SW1.1, SW2.1, SW3.1, SW4.1, SW5.1, SW6.1, SW7.1, SW8.1, TP7.1, U1.1 (GND), U3.4 (GND), U4.19 (TESTEN), U4.57 (GND), Y1.2, Y1.4
- net LDO_{VIN} renamed VBUS
- net VBUS: now also C1.1, C2.1, F1.2, LED1.1 (VDD), TP10.1, TP8.1, U1.3 (VI)
- new net: C6.1, U4.21 (XOUT), Y1.3
- new net: C5.1, U4.20 (XIN), Y1.1
- new net: TP4.1, U4.24 (SWCLK)
- new net: TP6.1, U4.25 (SWD)
- new net: TP3.1, U4.26 (RUN)
- new net: J1.B5 (CC2), R1.1
- new net: J1.A5 (CC1), R5.1
- new net $.GPIO0: SW6.2, U4.2 (GPIO0)
- new net $.GPIO7: U4.9 (GPIO7)
- new net +1V2: C10.1, C8.1, C9.1, TP2.1, U4.23 (DVDD), U4.45 (VREG_VOUT), U4.50 (DVDD)
- new net D+: R3.2, U4.47 (USB_DP)
- new net D-: R2.2, U4.46 (USB_DM)
- new net SCK: U3.6 (CLK), U4.52 (QSPI_SCLK)
- new net SD0: U3.5 (DI(IO0)), U4.53 (QSPI_SD0)
- new net SD1: U3.2 (DO(IO1)), U4.55 (QSPI_SD1)
- new net SD2: U3.3 (IO2), U4.54 (QSPI_SD2)
- new net SD3: U3.7 (IO3), U4.51 (QSPI_SD3)
- new net USB_VBUS: F1.1, J1.A4 (VBUS), J1.A9 (VBUS), J1.B4 (VBUS), J1.B9 (VBUS)
- new net USB_{DATA}+: J1.A6 (D+), J1.B6 (D+), R3.1
- new net USB_{DATA}-: J1.A7 (D-), J1.B7 (D-), R2.1
- new net ~{CS}: R6.1, TP12.1, U3.1 (~{CS}), U4.56 (QSPI_SS)
- no-connect marks 0 -> 4
Other:
- removed sheet Untitled Sheet
- removed sheet Untitled Sheet1
- removed sheet Untitled Sheet2
- removed sheet Untitled Sheet3
- removed sheet Untitled Sheet4
- moved on the sheet: J3A, J3B
