File: hardware/PicoGamePad_V3_0_0_A.kicad_sch (KiCad schematic)
At the start: 52 parts, among them J1 C116159, J3 RBP_GPIO_CONN, SW1 DOWN, SW2 START, SW3 LEFT, SW4 B, SW5 UP, SW6 A, SW7 RIGHT, SW8 SELECT, U1 ASM1117-3.3, U3 WQ25JVS, U4 RP2040, Y1 X322512MMB4SI

Commit message: 
Parts:
- removed JP1: Conn_01x02, Connector_PinSocket_2.54mm:PinSocket_1x02_P2.54mm_Vertical, symbol 4ms_Connector:Conn_01x02
- removed JP2: Conn_02x03, Connector_PinSocket_2.54mm:PinSocket_2x03_P2.54mm_Vertical, symbol 4ms_Connector:Conn_02x03
- removed R4: R, Resistor_SMD:R_0805_2012Metric, symbol Device:R
- removed R7: 1k, Resistor_SMD:R_0805_2012Metric, symbol Device:R
- added TP11: SWD_3V3, 0:Testpoint_Custom, symbol 4ms_Connector:TestPoint_Small
- added TP12: ~{CS}, 0:Testpoint_Custom, symbol Connector:TestPoint_Flag
- added TP3: RUN, 0:Testpoint_Custom, symbol 4ms_Connector:TestPoint_Small
- added TP4: SWCLK, 0:Testpoint_Custom, symbol 4ms_Connector:TestPoint_Small
- added TP6: SWD, 0:Testpoint_Custom, symbol 4ms_Connector:TestPoint_Small
- added TP7: RUN_GND, 0:Testpoint_Custom, symbol 4ms_Connector:TestPoint_Small
- U4: symbol 0:RP2040 -> MCU_RaspberryPi:RP2040
Connections:
- net X_{OUT} is gone; now on an unnamed net: U4.21 (XOUT)
- net +3V3: now also TP11.1
- net GND: now also TP7.1
- net ~{CS}: now also R6.1, TP12.1
- net SWCLK: no longer names the net of U4.24 (SWCLK)
- net SWCLK: now also TP4.1
- net SWD/SWDIO: no longer names the net of U4.25 (SWD)
- net SWD/SWDIO: now also TP6.1
- net X_{IN}: no longer names the net of C5.1, U4.20 (XIN), Y1.1
- net ~{RESET}/RUN: no longer names the net of U4.26 (RUN)
- net ~{RESET}/RUN: now also TP3.1
Other:
- moved on the sheet: C1, C10, C11, C12, C13, C14, C15, C16, C17, C18, C2, C3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
